File: hardware/kicad/hw/hw.kicad_sch (KiCad schematic)
At the start: 15 parts, among them J1 5V Power IN, SW3 InOut, SW4 OnOff, U1 XIAO-ESP32-S3-DIP, U2 SFH_4544, U3 TSOP4838

Commit message: checkin
Parts:
- added C3: 100nF, symbol Device:C
- added R6: 100, symbol Device:R
- C1, C2: value 1uF -> 10nF
Connections:
- net 3V3: now also R6.1; no longer ROT1.S2, SW3.2, SW4.2, U3.3 (VS)
- net GND: now also ROT1.S2, SW3.2, SW4.2, C3.2
- new net: C3.1, R6.2, U3.3 (VS)
Other:
- note added: "Bisherige Verbesserungsvorschläge: 1. Den IR Empfänger um 180 Grad drehen 2. Alle Buttons sollten Active LOW sein, ->OK jetzt sind sie active High. Das ist suboptimal, weil SW4 am GOPIO9 (STAPPING PIN) hängt. Der hat einen Pullup und deshalb wird er nie LOW 3. Die Beschriftungen im Layout der GPIOs ist falsch 4. 12V->5V DCDC-Converter integrieren, sicherung 4. Dem IR Receiver fehlt der Widerstand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"
