File: hardware/kicad/hw/hw.kicad_sch (KiCad schematic)
At the start: 17 parts, among them J1 5V Power IN, SW3 InOut, SW4 OnOff, U1 XIAO-ESP32-S3-DIP, U2 SFH_4544, U3 TSOP4838

Commit message: Vorwiderstand 100 Ohm
Parts:
- R1: value 330 -> 100
Other:
- note added: "Bisherige Verbesserungsvorschläge: 1. Den IR Empfänger um 180 Grad drehen 2. Alle Buttons sollten Active LOW sein, ->OK jetzt sind sie active High. Das ist suboptimal, weil SW4 am GOPIO9 (STAPPING PIN) hängt. Der hat einen Pullup und deshalb wird er nie LOW 3. Die Beschriftungen im Layout der GPIOs ist falsch 4. 12V->5V DCDC-Converter integrieren, sicherung ~200mA PTC, Diode gegen Verpolung 4. De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"
- note removed: "Bisherige Verbesserungsvorschläge: 1. Den IR Empfänger um 180 Grad drehen 2. Alle Buttons sollten Active LOW sein, ->OK jetzt sind sie active High. Das ist suboptimal, weil SW4 am GOPIO9 (STAPPING PIN) hängt. Der hat einen Pullup und deshalb wird er nie LOW 3. Die Beschriftungen im Layout der GPIOs ist falsch 4. 12V->5V DCDC-Converter integrieren, sicherung 4. Dem IR Receiver fehlt der Widerstand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"
Changed lines of the file:
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@@
 	(generator_version "9.0")
 	(paper "A4")
-	(text "Bisherige Verbesserungsvorschläge:\n\n1. Den IR Empfänger um 180 Grad drehen\n2. Alle Buttons sollten Active LOW sein, ->OK\njetzt sind sie active High. Das ist suboptimal, weil SW4 am GOPIO9 (STAPPING PIN)\n hängt. Der hat einen Pullup und deshalb wird er nie LOW\n3. Die Beschriftungen im Layout der GPIOs ist falsch\n\n4. 12V->5V DCDC-Converter integrieren, sicherung\n4. Dem IR Receiver fehlt der Widerstand und der Kondensator\n5. IR LED ev als SMD wählen, z.B. VSMY2940RGX01 https://www.vishay.com/docs/84583/vsmy2940rgx01.pdf\n6. Verpolungsschutz (Diode)\n7. Die Löscher zur Positionierung des Rotary Encoders könnten etwas kleiner gewählt werden.\n\nDer Vorwiderstand der IR LED soll nicht unter dem Display liegen"
+	(text "Bisherige Verbesserungsvorschläge:\n\n1. Den IR Empfänger um 180 Grad drehen\n2. Alle Buttons sollten Active LOW sein, ->OK\njetzt sind sie active High. Das ist suboptimal, weil SW4 am GOPIO9 (STAPPING PIN)\n hängt. Der hat einen Pullup und deshalb wird er nie LOW\n3. Die Beschriftungen im Layout der GPIOs ist falsch\n\n4. 12V->5V DCDC-Converter integrieren, sicherung ~200mA PTC, Diode gegen Verpolung\n4. Dem IR Receiver fehlt der Widerstand und der Kondensator\n5. IR LED ev als SMD wählen, z.B. VSMY2940RGX01 https://www.vishay.com/docs/84583/vsmy2940rgx01.pdf\n6. Verpolungsschutz (Diode)\n7. Die Löscher zur Positionierung des Rotary Encoders könnten etwas kleiner gewählt werden.\n\nDer Vorwiderstand der IR LED soll nicht unter dem Display liegen"
 		(exclude_from_sim no)
 		(at 127 129.54 0)
@@
 			)
 		)
-		(property "Value" "330"
+		(property "Value" "100"
 			(at 69.85 45.72 90)
 			(effects
