File: hardware/kicad/hw/hw.kicad_sch (KiCad schematic)
At the start: 17 parts, among them J1 5V Power IN, SW3 InOut, SW4 OnOff, U1 XIAO-ESP32-S3-DIP, U2 SFH_4544, U3 TSOP4838

Commit message: chec
Parts:
- removed U2: SFH_4544, SFH_4544:SFH213FA, symbol SFH_4544:SFH_4544
- added C4, C5: 47uF, CAP_EEEFK1V470P:CAP_EEEFK1V470P, symbol Device:C_Polarized
- added CBoot1, Cinx1: 100nF, Capacitor_SMD:C_0805_2012Metric, symbol Device:C
- added COut1, COut2: 10uF, Resistor_SMD:R_0805_2012Metric_Pad1.20x1.40mm_HandSolder, symbol Device:C
- added Cin1: 4.7uF, Capacitor_SMD:C_0805_2012Metric_Pad1.18x1.45mm_HandSolder, symbol Device:C
- added D1: RB168MM-40TFTR, RB168MM40TFTR:RB168MM40TFTR, symbol RB168MM-40TFTR:RB168MM-40TFTR
- added D2: SMBJ18A, DIONM5436X261N:DIONM5436X261N, symbol SMBJ18A:SMBJ18A
- added F1: 1206L025_24YR, FUSC3216X100N:FUSC3216X100N, symbol 1206L025_24YR:1206L025_24YR
- added L1: 15uH, SRN5040:SRN5040, symbol Device:L
- added L2: L_Ferrite, Inductor_SMD:L_1206_3216Metric_Pad1.22x1.90mm_HandSolder, symbol Device:L_Ferrite
- added LED1: VSMY2940RGX01, VSMY2940RGX01:VSMY2940RGX01, symbol VSMY2940RGX01:VSMY2940RGX01
- added PS1: LMR50410XDBVR, LMR50410XDBVR:SOT95P280X145-6N, symbol LMR50410XDBVR:LMR50410XDBVR
- added Rfbb1: 22.1k, Resistor_SMD:R_0805_2012Metric_Pad1.20x1.40mm_HandSolder, symbol Device:R
- added Rfbt1: 88.7k, Resistor_SMD:R_0805_2012Metric_Pad1.20x1.40mm_HandSolder, symbol Device:R
- added TP1: TestPoint, TestPoint:TestPoint_Pad_2.0x2.0mm, symbol Connector:TestPoint
- C3: footprint (none) -> Capacitor_SMD:C_0805_2012Metric
- J1: value 5V Power IN -> Power IN
- R6: footprint (none) -> Resistor_SMD:R_1206_3216Metric_Pad1.30x1.75mm_HandSolder
- U1: value XIAO-ESP32-S3-DIP -> XIAO-ESP32-C6-DIP
Connections:
- net GND: now also C4.2, C5.2, COut1.2, COut2.2, Cin1.2, Cinx1.2, D2.2 (A), LED1.1 (K), PS1.2 (GND), Rfbb1.2
- net at R1.2: now also LED1.2 (A); no longer U1.1 (GPIO1/D0/A0)
- net +12V: now reaches J1.1 (Pin_1)
- net +12V: now also F1.2; no longer U1.14 (VBUS)
- net at R1.1: now also U1.1 (D0)
- new net: C4.1, C5.1, D1.1 (K), D2.1 (K), L2.2
- new net: CBoot1.1, PS1.1 (CB)
- new net: CBoot1.2, L1.1, PS1.6 (SW)
- new net: D1.2 (A), F1.1
- new net: PS1.3 (FB), Rfbb1.1, Rfbt1.2
- new net: Cin1.1, Cinx1.1, L2.1, PS1.4 (EN), PS1.5 (VIN)
- new net +5V: COut1.1, COut2.1, L1.2, Rfbt1.1, TP1.1, U1.14 (5V)
Other:
- note added: "Bisherige Verbesserungsvorschläge: 1. Den IR Empfänger um 180 Grad drehen 2. Alle Buttons sollten Active LOW sein, ->OK jetzt sind sie active High. Das ist suboptimal, weil SW4 am GOPIO9 (STAPPING PIN) hängt. Der hat einen Pullup und deshalb wird er nie LOW 3. Die Beschriftungen im Layout der GPIOs ist falsch 4. 12V->5V DCDC-Converter integrieren, sicherung ~200mA PTC, Diode gegen Verpolung -> OK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"
- note removed: "Bisherige Verbesserungsvorschläge: 1. Den IR Empfänger um 180 Grad drehen 2. Alle Buttons sollten Active LOW sein, ->OK jetzt sind sie active High. Das ist suboptimal, weil SW4 am GOPIO9 (STAPPING PIN) hängt. Der hat einen Pullup und deshalb wird er nie LOW 3. Die Beschriftungen im Layout der GPIOs ist falsch 4. 12V->5V DCDC-Converter integrieren, sicherung ~200mA PTC, Diode gegen Verpolung 4. De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"
- moved on the sheet: R1

Commit message: changes
Parts:
- added TP2: TestPoint, TestPoint:TestPoint_Pad_2.0x2.0mm, symbol Connector:TestPoint
- C1, C2: footprint Capacitor_SMD:C_1206_3216Metric_Pad1.33x1.80mm_HandSolder -> Capacitor_SMD:C_0805_2012Metric_Pad1.18x1.45mm_HandSolder
- C3, CBoot1, Cinx1: footprint Capacitor_SMD:C_0805_2012Metric -> Capacitor_SMD:C_0805_2012Metric_Pad1.18x1.45mm_HandSolder
- R1, R2, R3, R4, R5, R6: footprint Resistor_SMD:R_1206_3216Metric_Pad1.30x1.75mm_HandSolder -> Resistor_SMD:R_0805_2012Metric_Pad1.20x1.40mm_HandSolder
Connections:
- net at C4.1, C5.1, D1.1 (K)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: now also TP2.1
Changed lines of the file:
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@@
 	)
 	(junction
+		(at 91.186 172.72)
+		(diameter 0)
+		(color 0 0 0 0)
+	)
+	(junction
 		(at 81.28 172.72)
 		(diameter 0)
@@
 	(wire
 		(pts
+			(xy 91.186 172.72) (xy 95.25 172.72)
+		)
+		(stroke
+			(width 0)
+			(type default)
+		)
+	)
+	(wire
+		(pts
 			(xy 45.72 123.19) (xy 25.4 123.19)
 		)
@@
 	(wire
 		(pts
-			(xy 87.63 172.72) (xy 95.25 172.72)
+			(xy 87.63 172.72) (xy 91.186 172.72)
 		)
 		(stroke
@@
 			)
 		)
-		(property "Footprint" "Capacitor_SMD:C_0805_2012Metric"
+		(property "Footprint" "Capacitor_SMD:C_0805_2012Metric_Pad1.18x1.45mm_HandSolder"
 			(at 39.37 148.8948 0)
 			(effects
@@
 			)
 		)
-		(property "Footprint" "Resistor_SMD:R_1206_3216Metric_Pad1.30x1.75mm_HandSolder"
+		(property "Footprint" "Resistor_SMD:R_0805_2012Metric_Pad1.20x1.40mm_HandSolder"
 			(at 49.022 118.11 90)
 			(effects
@@
 			)
 		)
-		(property "Footprint" "Resistor_SMD:R_1206_3216Metric_Pad1.30x1.75mm_HandSolder"
+		(property "Footprint" "Resistor_SMD:R_0805_2012Metric_Pad1.20x1.40mm_HandSolder"
 			(at 69.85 47.752 90)
 			(effects
@@
 			)
 		)
-		(property "Footprint" "Resistor_SMD:R_1206_3216Metric_Pad1.30x1.75mm_HandSolder"
+		(property "Footprint" "Resistor_SMD:R_0805_2012Metric_Pad1.20x1.40mm_HandSolder"
 			(at 38.1 116.078 90)
 			(effects
@@
 			)
 		)
-		(property "Footprint" "Capacitor_SMD:C_0805_2012Metric"
+		(property "Footprint" "Capacitor_SMD:C_0805_2012Metric_Pad1.18x1.45mm_HandSolder"
 			(at 154.6352 64.77 0)
 			(effects
@@
 			)
 		)
-		(property "Footprint" "Capacitor_SMD:C_1206_3216Metric_Pad1.33x1.80mm_HandSolder"
+		(property "Footprint" "Capacitor_SMD:C_0805_2012Metric_Pad1.18x1.45mm_HandSolder"
 			(at 46.6852 130.81 0)
 			(effects
@@
 			)
 		)
-		(property "Footprint" "Resistor_SMD:R_1206_3216Metric_Pad1.30x1.75mm_HandSolder"
+		(property "Footprint" "Resistor_SMD:R_0805_2012Metric_Pad1.20x1.40mm_HandSolder"
 			(at 58.42 116.078 90)
 			(effects
@@
 			)
 		)
-		(property "Footprint" "Resistor_SMD:R_1206_3216Metric_Pad1.30x1.75mm_HandSolder"
+		(property "Footprint" "Resistor_SMD:R_0805_2012Metric_Pad1.20x1.40mm_HandSolder"
 			(at 148.59 58.928 90)
 			(effects
@@
 			)
 		)
-		(property "Footprint" "Resistor_SMD:R_1206_3216Metric_Pad1.30x1.75mm_HandSolder"
+		(property "Footprint" "Resistor_SMD:R_0805_2012Metric_Pad1.20x1.40mm_HandSolder"
 			(at 43.942 118.11 90)
 			(effects
@@
 	)
 	(symbol
+		(lib_id "Connector:TestPoint")
+		(at 91.186 172.72 0)
+		(unit 1)
+		(exclude_from_sim no)
+		(in_bom yes)
+		(on_board yes)
+		(dnp no)
+		(fields_autoplaced yes)
+		(property "Reference" "TP2"
+			(at 92.71 168.1479 0)
+			(effects
+				(font
+					(size 1.27 1.27)
+				)
+				(justify left)
+			)
+		)
+		(property "Value" "TestPoint"
+			(at 92.71 170.6879 0)
+			(effects
+				(font
+					(size 1.27 1.27)
+				)
+				(justify left)
+			)
+		)
+		(property "Footprint" "TestPoint:TestPoint_Pad_2.0x2.0mm"
+			(at 96.266 172.72 0)
+			(effects
+				(font
+					(size 1.27 1.27)
+				)
+				(hide yes)
+			)
+		)
+		(property "Datasheet" "~"
+			(at 96.266 172.72 0)
+			(effects
+				(font
+					(size 1.27 1.27)
+				)
+				(hide yes)
+			)
+		)
+		(property "Description" "test point"
+			(at 91.186 172.72 0)
+			(effects
+				(font
+					(size 1.27 1.27)
+				)
+				(hide yes)
+			)
+		)
+		(pin "1"
+		)
+		(instances
+			(project ""
+				(path "/204b0454-dab1-43cb-9d67-c9c471af0977"
+					(reference "TP2")
+					(unit 1)
+				)
+			)
+		)
+	)
+	(symbol
 		(lib_id "Device:C")
 		(at 152.4 168.91 0)
@@
 			)
 		)
-		(property "Footprint" "Capacitor_SMD:C_0805_2012Metric"
+		(property "Footprint" "Capacitor_SMD:C_0805_2012Metric_Pad1.18x1.45mm_HandSolder"
 			(at 54.3052 184.15 0)
 			(effects
@@
 			)
 		)
-		(property "Footprint" "Capacitor_SMD:C_1206_3216Metric_Pad1.33x1.80mm_HandSolder"
+		(property "Footprint" "Capacitor_SMD:C_0805_2012Metric_Pad1.18x1.45mm_HandSolder"
 			(at 51.7652 130.81 0)
 			(effects
