File: hardware/kicad/hw/hw.kicad_pcb (KiCad board)
At the start: 2 copper layers, 75.7 x 75.7 mm, 15 parts, among them J1 5V Power IN, SW3 InOut, SW4 OnOff, U1 XIAO-ESP32-S3-DIP, U2 SFH_4544, U3 TSOP4838

Commit message: chec
Parts:
- removed U2: SFH_4544, SFH_4544:SFH213FA
- added C3: 100nF, Capacitor_SMD:C_0805_2012Metric, F.Cu at (133.3, 116.2)
- added C4: 47uF, CAP_EEEFK1V470P:CAP_EEEFK1V470P, F.Cu at (149.9, 73.9)
- added C5: 47uF, CAP_EEEFK1V470P:CAP_EEEFK1V470P, F.Cu at (162.9, 74.7)
- added CBoot1: 100nF, Capacitor_SMD:C_0805_2012Metric, F.Cu at (141.7, 91.3)
- added COut1: 10uF, Resistor_SMD:R_0805_2012Metric_Pad1.20x1.40mm_HandSolder, F.Cu at (158.5, 89.5)
- added COut2: 10uF, Resistor_SMD:R_0805_2012Metric_Pad1.20x1.40mm_HandSolder, F.Cu at (156.5, 89.5)
- added Cin1: 4.7uF, Capacitor_SMD:C_0805_2012Metric_Pad1.18x1.45mm_HandSolder, F.Cu at (147.4, 89.5)
- added Cinx1: 100nF, Capacitor_SMD:C_0805_2012Metric, F.Cu at (148.2, 94.4)
- added D1: RB168MM-40TFTR, RB168MM40TFTR:RB168MM40TFTR, F.Cu at (180.6, 75.2)
- added D2: SMBJ18A, DIONM5436X261N:DIONM5436X261N, F.Cu at (174.2, 78.2)
- added F1: 1206L025_24YR, FUSC3216X100N:FUSC3216X100N, F.Cu at (181.2, 69.7)
- added L1: 15uH, SRN5040:SRN5040, F.Cu at (154.4, 94.2)
- added L2: L_Ferrite, Inductor_SMD:L_1206_3216Metric_Pad1.22x1.90mm_HandSolder, F.Cu at (144.5, 85.6)
- added LED1: VSMY2940RGX01, VSMY2940RGX01:VSMY2940RGX01, F.Cu at (142.5, 80.1)
- added PS1: LMR50410XDBVR, LMR50410XDBVR:SOT95P280X145-6N, F.Cu at (144.9, 93.2)
- added R6: 100, Resistor_SMD:R_1206_3216Metric_Pad1.30x1.75mm_HandSolder, F.Cu at (136.1, 118.1)
- added Rfbb1: 22.1k, Resistor_SMD:R_0805_2012Metric_Pad1.20x1.40mm_HandSolder, F.Cu at (148.1, 99.7)
- added Rfbt1: 88.7k, Resistor_SMD:R_0805_2012Metric_Pad1.20x1.40mm_HandSolder, F.Cu at (150.4, 99.7)
- added TP1: TestPoint, TestPoint:TestPoint_Pad_2.0x2.0mm, F.Cu at (153.5, 87.8)
- C1, C2: value 1uF -> 10nF
- J1: value 5V Power IN -> Power IN
- R1: value 330 -> 100
- U1: value XIAO-ESP32-S3-DIP -> XIAO-ESP32-C6-DIP
- moved R1 20.6 mm to (136.9, 81.8), turned to 90 degrees
- moved C2 10.9 mm to (127.9, 89.2)
- moved R2 6.67 mm to (123.1, 90.0)
- moved C1 5.60 mm to (123.1, 79.0), turned to 90 degrees
- moved R3 2.74 mm to (123.1, 84.7)
- moved R5 2.03 mm to (140.0, 85.6)
- moved R4 1.27 mm to (133.6, 86.6)
- moved J1 0.10 mm to (181.1, 63.3)
- moved ROT1 0.10 mm to (132.0, 67.1)
- moved U3 0.10 mm to (124.8, 121.4)
- moved OLED1 0.10 mm to (154.5, 67.7)
- moved SW3 0.10 mm to (170.2, 64.7)
- moved SW4 0.10 mm to (170.3, 74.0)
- moved U1 0.10 mm to (128.3, 103.8)
Connections:
- J1 pad 1: Net-(J1-Pin_1) -> +12V
- R1 pad 1: Net-(U2-A) -> Net-(U1-D0)
- R1 pad 2: Net-(U1-GPIO1/D0/A0) -> Net-(LED1-A)
- ROT1 pad S2: /3V3 -> GND
- SW3 pad 2: /3V3 -> GND
- SW4 pad 2: /3V3 -> GND
- U1 pad 1: Net-(U1-GPIO1/D0/A0) -> Net-(U1-D0)
- U1 pad 14: Net-(J1-Pin_1) -> +5V
- U3 pad 3: /3V3 -> Net-(U3-VS)
Routing:
- net Net-(J1-Pin_1): track 107.9 -> 0.00 mm
- net Net-(D1-K): track 0.00 -> 63.5 mm, vias 0 -> 2
- net Net-(U1-GPIO1/D0/A0): track 53.5 -> 0.00 mm, vias 2 -> 0
- net +5V: track 0.00 -> 52.6 mm, vias 0 -> 4
- net /3V3: track 135.3 -> 88.5 mm, vias 2 -> 4
- net Net-(U1-D0): track 0.00 -> 37.6 mm
- net Net-(U1-D9): track 57.6 -> 89.0 mm, vias 3 -> 1
- net Net-(U1-D2): track 63.8 -> 33.0 mm
- net Net-(U3-VS): track 0.00 -> 21.7 mm
- net Net-(PS1-EN): track 0.00 -> 20.1 mm, vias 0 -> 2
- net Net-(PS1-SW): track 0.00 -> 16.8 mm, vias 0 -> 3
- net Net-(PS1-FB): track 0.00 -> 16.2 mm, vias 0 -> 4
- net Net-(OLED1-SDA): track 82.9 -> 67.4 mm, vias 0 -> 2
- net GND: track 28.4 -> 41.6 mm, vias 3 -> 14
- net Net-(U1-D8): track 34.4 -> 21.6 mm, vias 0 -> 2
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Other:
- outline, holes or cut-outs redrawn
- board text added: "."

Commit message: changes
Parts:
- added TP2: TestPoint, TestPoint:TestPoint_Pad_2.0x2.0mm, F.Cu at (156.3, 74.2)
- C1, C2: footprint Capacitor_SMD:C_1206_3216Metric_Pad1.33x1.80mm_HandSolder -> Capacitor_SMD:C_0805_2012Metric_Pad1.18x1.45mm_HandSolder
- C3, CBoot1, Cinx1: footprint Capacitor_SMD:C_0805_2012Metric -> Capacitor_SMD:C_0805_2012Metric_Pad1.18x1.45mm_HandSolder
- R1, R2, R3, R4, R5, R6: footprint Resistor_SMD:R_1206_3216Metric_Pad1.30x1.75mm_HandSolder -> Resistor_SMD:R_0805_2012Metric_Pad1.20x1.40mm_HandSolder
- moved R5 18.7 mm to (121.5, 82.9), turned to -90 degrees
- moved R2 11.5 mm to (132.2, 83.1)
- moved C1 9.55 mm to (128.3, 87.0), turned to -90 degrees
- moved R4 9.16 mm to (125.2, 82.9)
- moved R3 5.46 mm to (128.3, 83.1), turned to -90 degrees
- moved C2 3.43 mm to (125.2, 87.0), turned to -90 degrees
- moved C3 2.10 mm to (132.5, 118.1)
- moved Rfbt1 1.02 mm to (151.4, 99.7)
- moved R6 0.38 mm to (135.8, 118.1), turned to -90 degrees
Routing:
- net Net-(U1-D10): track 67.4 -> 86.7 mm, vias 6 -> 4
- net Net-(U1-D9): track 89.0 -> 75.7 mm, vias 1 -> 3
- net Net-(U1-D3): track 28.9 -> 42.1 mm, vias 4 -> 2
- net Net-(R2-Pad2): track 42.6 -> 31.0 mm
- net Net-(U3-VS): track 21.7 -> 12.1 mm
- net Net-(R4-Pad1): track 35.9 -> 28.3 mm, vias 2 -> 0
- net /3V3: track 88.5 -> 92.0 mm, vias 4 -> 6
- net Net-(U1-D2): track 33.0 -> 31.2 mm
- net Net-(D1-K): track 63.5 -> 64.9 mm
- net Net-(PS1-FB): track 16.2 -> 17.2 mm
- net GND: track 41.6 -> 40.8 mm
- net Net-(U1-D8): track 21.6 -> 22.3 mm, vias 2 -> 4
Other:
- board text added: "B"
